File: ASD2431.brd (EAGLE design)
At the start: 28.3 x 26.3 mm, 30 parts, among them J1 EVP-ANDA1A, J2 DF12-32-DS, J3 EVP-ANDA1A, J4 EVP-ANDA1A, J5 EVP-ANDA1A, U1 XC6210B33, U2 TXB0104, U3 UG-9664HDDAG01, U4 FAN5331SX, U5 SX1505I087TRT

Commit message: Update to rev 5
Parts:
- added C7: 0.1uF, tinycircuits:C0402
- added J10, J11, J6, J7, J8, J9: (no value), tinycircuits:TEST_POINT_1MM
- added R10, R11: 0.0, tinycircuits:0402
- C2, C5: value 10uF -> 1uF; device tinycircuits:C0805 -> tinycircuits:C0402
- U1: value XC6210B33 -> XC6217A33
- moved C6 24.0 mm to (20.6, 6.20), turned to 0 degrees
- moved C2 19.3 mm to (17.5, 9.55), turned to 180 degrees
- moved C15 3.10 mm to (8.75, 26.1)
- moved C5 2.49 mm to (19.8, 9.55), turned to 180 degrees
- moved C1 2.20 mm to (19.8, 8.50), turned to 180 degrees
- moved D1 0.45 mm to (24.6, 6.11)
- moved U1 0.40 mm to (16.9, 7.42)
- moved U5 0.36 mm to (12.2, 7.95)
- moved R7 0.36 mm to (15.2, 9.55)
- moved R1 0.35 mm to (22.2, 7.63)
- moved C9 0.35 mm to (22.2, 8.61)
- moved R2 0.30 mm to (22.2, 9.55)
- moved L1 0.21 mm to (27.5, 7.23)
- moved R4 0.15 mm to (8.65, 6.65)
- moved R5 0.15 mm to (8.65, 5.85)
Connections:
- removed net N$16: U3.16
- removed net N$17: U3.17
- removed net N$18: U3.18
- removed net N$19: U3.19
- removed net N$20: U3.20
- removed net N$9: U5.9
- new net INT: R10.1, R11.1, U5.11
- new net SHDN: U4.4, U5.9
- net +12V: now also J11.P$1
- net CS#: now also J6.P$1
- net D/C#: now also J8.P$1
- net GND: now also C7.2, U1.4, U3.16, U3.17, U3.18, U3.19, U3.20
- net IO2: now also R10.2
- net IO3: now also R11.2
- net RES#: now also J7.P$1
- net SCLK: now also J9.P$1
- net SDIN: now also J10.P$1
- net VCC: now also C7.1; no longer U4.4
Routing:
- net GND: track 17.2 -> 65.9 mm, vias 16 -> 20
- net INT: track 0.00 -> 18.1 mm, vias 0 -> 2
- net SHDN: track 0.00 -> 15.5 mm, vias 0 -> 2
- net IO3: track 0.00 -> 13.3 mm
- net IO2: track 0.00 -> 11.5 mm
- net +12V: track 47.5 -> 41.4 mm, vias 2 -> 4
- net D/C#: track 3.26 -> 9.19 mm
- net SDIN: track 2.87 -> 8.69 mm
- net SCLK: track 2.63 -> 8.21 mm
- net CS#: track 4.20 -> 9.64 mm
- net VCC: track 71.7 -> 67.0 mm, vias 2 -> 4
- net RES#: track 42.2 -> 45.0 mm
- net N$6: track 11.0 -> 12.6 mm
- net N$2: track 4.18 -> 2.72 mm
- net VCC_3V3: track 48.8 -> 49.6 mm
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Other:
- board text added: "5"
- board text added: "ASD2431 - Rev5"
- board text removed: "4"
- board text removed: "ASD2431 - Rev4"
