File: ASD2431.sch (EAGLE design)
At the start: 29 parts, among them J1 EVP-ANDA1A, J2 DF12-32-DS, J3 EVP-ANDA1A, J4 EVP-ANDA1A, J5 EVP-ANDA1A, U1 XC6210B33, U2 TXB0104, U3 UG-9664HDDAG01, U4 FAN5331SX, U5 SX1505I087TRT

Commit message: Update to rev 5
Parts:
- added C7: 0.1uF, tinycircuits:AS-ITM-00008
- added J10, J11, J6, J7, J8, J9: (no value), tinycircuits:TEST_POINT
- added R10, R11: 0.0, tinycircuits:AS-ITM-00076
- C2: value 10uF -> 1uF; device tinycircuits:AS-ITM-00045 -> tinycircuits:AS-ITM-00105; PARTNO AS-ITM-00045 -> AS-ITM-00105; VALUE 10uF -> 1uF
- C5: value 10uF -> 1uF; device tinycircuits:AS-ITM-00045 -> tinycircuits:AS-ITM-00105; PARTNO (none) -> AS-ITM-00105; VALUE (none) -> 1uF
- U1: value XC6210B33 -> XC6217A33; device tinycircuits:AS-ITM-00046 -> tinycircuits:AS-ITM-00249; PARTNO (none) -> AS-ITM-00249; VALUE (none) -> XC6217A33
Connections:
- removed net N$16: U3.D3
- removed net N$17: U3.D4
- removed net N$18: U3.D5
- removed net N$19: U3.D6
- removed net N$20: U3.D7
- removed net N$9: U5.IO2
- new net INT: R10.1, R11.1, U5.NINT
- new net SHDN: U4.SHDN, U5.IO2
- net +12V: now also J11.1
- net CS#: now also J6.1
- net D/C#: now also J8.1
- net GND: now also C7.2, U1.NC/GO, U3.D3, U3.D4, U3.D5, U3.D6, U3.D7
- net IO2: now also R10.2
- net IO3: now also R11.2
- net RES#: now also J7.1
- net SCLK: now also J9.1
- net SDIN: now also J10.1
- net VCC: now also C7.1; no longer U4.SHDN
Other:
- note added: "5"
- note removed: "4"
- moved on the sheet: C15, J1, J3, J4, J5, R3, R8, R9, U2, U3
