File: design_files/ASD2431.sch (EAGLE design)
At the start: 38 parts, among them J1 EVP-ANDA1A, J2 DF12-32-DS, J3 EVP-ANDA1A, J4 EVP-ANDA1A, J5 EVP-ANDA1A, U1 XC6217A33, U2 TXB0104, U3 UG-9664HDDAG01, U4 FAN5331SX, U5 SX1505I087TRT

Commit message: update files
Parts:
- removed C15: 4.7uF, tinycircuits:AS-ITM-00232
- added C8: 100pF, tinycircuits:AS-ITM-00148
- C9: value 180pF -> 4.7uF; device tinycircuits:AS-ITM-00243 -> tinycircuits:AS-ITM-00232; PARTNO AS-ITM-00243 -> AS-ITM-00232; VALUE 180pF -> F931D475MAA
- J1: value EVP-ANDA1A -> DF12-32-DS; device tinycircuits:AS-ITM-00236 -> tinycircuits:AS-ITM-00012; PARTNO AS-ITM-00236 -> AS-ITM-00012; VALUE PTS840 GKP -> DF12-32-DS
- J2: value DF12-32-DS -> EVP-ANDA1A; device tinycircuits:AS-ITM-00012 -> tinycircuits:AS-ITM-00236; PARTNO AS-ITM-00012 -> AS-ITM-00236; VALUE DF12-32-DS -> PTS840 GKP
- R1: value 100K -> 200K; device tinycircuits:AS-ITM-00004 -> tinycircuits:AS-ITM-00178; PARTNO (none) -> AS-ITM-00178; VALUE (none) -> 200K
- R2: value 10.0K -> 22.0K; device tinycircuits:AS-ITM-00032 -> tinycircuits:AS-ITM-00147; PARTNO (none) -> AS-ITM-00147; VALUE (none) -> 22K
- R3: value 1.00M -> 1.2M; device tinycircuits:AS-ITM-00005 -> tinycircuits:AS-ITM-00280; PARTNO (none) -> AS-ITM-00280; VALUE (none) -> 1.2M
Connections:
- net +12V: now also C8.1; no longer C9.1
- net +3V3: now also J1.6; no longer J2.6
- net +5V: now also J1.8; no longer J2.8
- net AD0: now also J1.11; no longer J2.11
- net AD1: now also J1.9; no longer J2.9
- net AD2: now also J1.7; no longer J2.7
- net AD3: now also J1.5; no longer J2.5
- net AD4/SDA: now also J1.3; no longer J2.3
- net AD5/SCL: now also J1.1; no longer J2.1
- net AREF: now also J1.13; no longer J2.13
- net BTN0: now also J2.1; no longer J1.1
- net BTN2: now also J4.1; no longer J5.1
- net BTN3: now also J5.1; no longer J4.1
- net GND: now also C9.2, J1.12, J1.14, J2.2; no longer C15.2, J1.2, J2.12, J2.14
- net IO0: now also J1.24; no longer J2.24
- net IO1: now also J1.26; no longer J2.26
- net IO2: now also J1.28; no longer J2.28
- net IO3: now also J1.30; no longer J2.30
- net IO4: now also J1.32; no longer J2.32
- net IO5: now also J1.31; no longer J2.31
- net IO6: now also J1.29; no longer J2.29
- net IO7: now also J1.27; no longer J2.27
- net IO8: now also J1.25; no longer J2.25
- net IO9: now also J1.23; no longer J2.23
- net MISO: now also J1.17; no longer J2.17
- net MOSI: now also J1.19; no longer J2.19
- net N$3: now also C8.2; no longer C9.2
- net N$7: now also C9.1; no longer C15.1
- net RESET: now also J1.22; no longer J2.22
- net RSV0: now also J1.20; no longer J2.20
- net RSV1: now also J1.18; no longer J2.18
- net RSV2: now also J1.16; no longer J2.16
- net SCK: now also J1.15; no longer J2.15
- net SS: now also J1.21; no longer J2.21
- net VBATT: now also J1.4; no longer J2.4
- net VCC: now also J1.2; no longer J2.2
- net VIN: now also J1.10; no longer J2.10
Other:
- note added: "6"
- note added: "Default: Address 0 R5 populated, R4 unpopulated"
- note added: "Hand Populated: U3"
- note added: "Hand Soldered: -"
- note added: "Non Populated: R4, R10, R11"
- note added: "Notes: -"
- note added: "Optional interrupt from GPIO, unpopulated by default"
- note added: "Variant: Standard - R"
- note removed: "5"
- moved on the sheet: C4, C9, J4, J5
